File: ble/ble.kicad_pcb (KiCad board)
At the start: 4 copper layers, 27 x 46 mm, 61 parts, among them J1 I2C, J2 SPI, J3 ADC, J4 ANATEST, J5 USB_OTG, U1 TLV62568DBV, U2 BLUENRG-232, U3 FT230XQ, U4 BALF-NRG-02D3, U5 EAST1616RGBA8, Y1 32.768kHz, Y2 32MHz

Commit message: report
Parts:
- J2: value SPI -> IO; footprint Connector_PinHeader_2.54mm:PinHeader_1x04_P2.54mm_Vertical -> Connector_PinHeader_2.54mm:PinHeader_1x02_P2.54mm_Vertical
- moved J2 5.12 mm to (102.5, 121.5)
Connections:
- net /SPI_MOSI renamed /DIO10
- J2 pad 1: /SPI_CLK -> /DIO9
- U2 pad 2: /SPI_MISO -> /DIO9
- U2 pad 3: /SPI_CLK -> /UART_RX
- U2 pad 32: /SPI_CS -> /UART_TX
- U2 pad 7: /UART_RX -> unconnected-(U2-DIO5-Pad7)
- U2 pad 8: /UART_TX -> unconnected-(U2-DIO4-Pad8)
Routing:
- net /SPI_CLK: track 14.6 -> 0.00 mm, vias 1 -> 0
- net /SPI_MISO: track 11.4 -> 0.00 mm, vias 1 -> 0
- net /DIO9: track 0.00 -> 11.3 mm, vias 0 -> 1
- net /SPI_CS: track 9.11 -> 0.00 mm, vias 1 -> 0
- net /UART_TX: track 16.2 -> 20.5 mm
- net /DIO10: track 12.4 -> 9.50 mm
- net /UART_RX: track 20.2 -> 22.2 mm
- net /UART_RTS: track 27.8 -> 26.0 mm
- net GND: track 32.3 -> 32.2 mm, vias 68 -> 72
Other:
- board text added: "ADC2 ADC1"
- board text added: "ANATEST1 ANATEST0"
- board text added: "DIO10 DIO9"
- board text added: "SDA SCL"
