File: ble/ble.kicad_sch (KiCad schematic)
At the start: 61 parts, among them J1 I2C, J2 SPI, J3 ADC, J4 ANATEST, J5 USB_OTG, U1 TLV62568DBV, U2 BLUENRG-232, U3 FT230XQ, U4 BALF-NRG-02D3, U5 EAST1616RGBA8, Y1 32.768kHz, Y2 32MHz

Commit message: report
Parts:
- removed J2: SPI, Connector_PinHeader_2.54mm:PinHeader_1x04_P2.54mm_Vertical, symbol Connector_Generic:Conn_01x04
- added J2: IO, Connector_PinHeader_2.54mm:PinHeader_1x02_P2.54mm_Vertical, symbol Connector_Generic:Conn_01x02
Connections:
- net SPI_CLK is gone; now on net UART_RX: U2.3 (DIO8)
- net SPI_CS is gone; now on net UART_TX: U2.32 (DIO11)
- net UART_RX: no longer U2.7 (DIO5)
- net UART_TX: no longer U2.8 (DIO4)
- net SPI_MISO renamed DIO9
- net DIO9: now also J2.1 (Pin_1)
- net SPI_MOSI renamed DIO10
- net DIO10: now also J2.2 (Pin_2)
Changed lines of the file:
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@@
-    (stroke (width 0) (type default))
-  )
-  (wire (pts (xy 121.92 123.19) (xy 132.08 123.19))
     (stroke (width 0) (type default))
   )
@@
     (stroke (width 0) (type default))
   )
-  (wire (pts (xy 35.56 167.64) (xy 24.13 167.64))
-    (stroke (width 0) (type default))
-  )
   (wire (pts (xy 54.61 33.02) (xy 64.77 33.02))
     (stroke (width 0) (type default))
@@
     (stroke (width 0) (type default))
   )
-  (wire (pts (xy 121.92 120.65) (xy 132.08 120.65))
-    (stroke (width 0) (type default))
-  )
   (wire (pts (xy 115.57 167.64) (xy 113.03 167.64))
     (stroke (width 0) (type default))
@@
   )
   (wire (pts (xy 207.01 97.79) (xy 207.01 96.52))
-    (stroke (width 0) (type default))
-  )
-  (wire (pts (xy 35.56 170.18) (xy 24.13 170.18))
     (stroke (width 0) (type default))
   )
@@
     (effects (font (size 1.27 1.27)) (justify right bottom))
   )
-  (label "SPI_CLK" (at 35.56 162.56 180) (fields_autoplaced)
+  (label "DIO9" (at 35.56 162.56 180) (fields_autoplaced)
     (effects (font (size 1.27 1.27)) (justify right bottom))
   )
@@
     (effects (font (size 1.27 1.27)) (justify left bottom))
   )
-  (label "SPI_CS" (at 35.56 170.18 180) (fields_autoplaced)
-    (effects (font (size 1.27 1.27)) (justify right bottom))
-  )
   (label "NRESET" (at 172.72 55.88 0) (fields_autoplaced)
     (effects (font (size 1.27 1.27)) (justify left bottom))
@@
     (effects (font (size 1.27 1.27)) (justify left bottom))
   )
-  (label "UART_TX" (at 121.92 120.65 0) (fields_autoplaced)
-    (effects (font (size 1.27 1.27)) (justify left bottom))
-  )
   (label "BOOT" (at 121.92 128.27 0) (fields_autoplaced)
     (effects (font (size 1.27 1.27)) (justify left bottom))
@@
     (effects (font (size 1.27 1.27)) (justify right bottom))
   )
-  (label "SPI_MOSI" (at 189.23 102.87 180) (fields_autoplaced)
-    (effects (font (size 1.27 1.27)) (justify right bottom))
-  )
-  (label "UART_RX" (at 121.92 123.19 0) (fields_autoplaced)
-    (effects (font (size 1.27 1.27)) (justify left bottom))
-  )
-  (label "SPI_MOSI" (at 35.56 165.1 180) (fields_autoplaced)
+  (label "DIO10" (at 189.23 102.87 180) (fields_autoplaced)
+    (effects (font (size 1.27 1.27)) (justify right bottom))
+  )
+  (label "DIO10" (at 35.56 165.1 180) (fields_autoplaced)
     (effects (font (size 1.27 1.27)) (justify right bottom))
   )
@@
     (effects (font (size 1.27 1.27)) (justify right bottom))
   )
-  (label "SPI_CS" (at 189.23 105.41 180) (fields_autoplaced)
+  (label "UART_TX" (at 189.23 105.41 180) (fields_autoplaced)
     (effects (font (size 1.27 1.27)) (justify right bottom))
   )
@@
     (effects (font (size 1.27 1.27)) (justify right bottom))
   )
-  (label "SPI_MISO" (at 35.56 167.64 180) (fields_autoplaced)
-    (effects (font (size 1.27 1.27)) (justify right bottom))
-  )
   (label "I2C_SCL" (at 189.23 107.95 180) (fields_autoplaced)
     (effects (font (size 1.27 1.27)) (justify right bottom))
@@
     (effects (font (size 1.27 1.27)) (justify left bottom))
   )
-  (label "SPI_MISO" (at 189.23 100.33 180) (fields_autoplaced)
+  (label "DIO9" (at 189.23 100.33 180) (fields_autoplaced)
     (effects (font (size 1.27 1.27)) (justify right bottom))
   )
@@
     (effects (font (size 1.27 1.27)) (justify left bottom))
   )
-  (label "SPI_CLK" (at 121.92 130.81 0) (fields_autoplaced)
+  (label "UART_RX" (at 121.92 130.81 0) (fields_autoplaced)
     (effects (font (size 1.27 1.27)) (justify left bottom))
   )
@@
     )
   )
-  (symbol (lib_id "Connector_Generic:Conn_01x04") (at 19.05 165.1 0) (mirror y) (unit 1)
-    (in_bom no) (on_board yes) (dnp no) (fields_autoplaced)
-    (property "Reference" "J2" (at 19.05 157.48 0)
-      (effects (font (size 1.27 1.27)))
-    )
-    (property "Value" "SPI" (at 19.05 160.02 0)
-      (effects (font (size 1.27 1.27)))
-    )
-    (property "Footprint" "Connector_PinHeader_2.54mm:PinHeader_1x04_P2.54mm_Vertical" (at 19.05 165.1 0)
-      (effects (font (size 1.27 1.27)) hide)
-    )
-    (property "Datasheet" "~" (at 19.05 165.1 0)
-      (effects (font (size 1.27 1.27)) hide)
-    )
-    (property "MPN" "" (at 19.05 165.1 0)
-      (effects (font (size 1.27 1.27)) hide)
-    )
-    (property "Item #" "" (at 19.05 165.1 0)
-      (effects (font (size 1.27 1.27)) hide)
-    )
-    (property "Description" "" (at 19.05 165.1 0)
-      (effects (font (size 1.27 1.27)) hide)
-    )
-    (property "Package/Footprint" "" (at 19.05 165.1 0)
-      (effects (font (size 1.27 1.27)) hide)
-    )
-    (property "Type" "Thru-hole" (at 19.05 165.1 0)
-      (effects (font (size 1.27 1.27)) hide)
-    )
-    (property "Your Instructions / Notes" "" (at 19.05 165.1 0)
-      (effects (font (size 1.27 1.27)) hide)
-    )
-    (pin "1")
-    (pin "2")
-    (pin "3")
-    (pin "4")
-    (instances
-      (project "ble"
-        (path "/a75a1d04-4959-44a9-a64e-65228c5b9ff4"
-          (reference "J2") (unit 1)
-        )
-      )
-    )
-  )
   (symbol (lib_id "Device:C_Small") (at 97.79 38.1 0) (unit 1)
     (in_bom yes) (on_board yes) (dnp no) (fields_autoplaced)
@@
         )
       )
+    )
+  )
+  (symbol (lib_id "Connector_Generic:Conn_01x02") (at 19.05 162.56 0) (mirror y) (unit 1)
+    (in_bom no) (on_board yes) (dnp no) (fields_autoplaced)
+    (property "Reference" "J2" (at 19.05 157.48 0)
+      (effects (font (size 1.27 1.27)))
+    )
+    (property "Value" "IO" (at 19.05 160.02 0)
+      (effects (font (size 1.27 1.27)))
+    )
+    (property "Footprint" "Connector_PinHeader_2.54mm:PinHeader_1x02_P2.54mm_Vertical" (at 19.05 162.56 0)
+      (effects (font (size 1.27 1.27)) hide)
+    )
+    (property "Datasheet" "~" (at 19.05 162.56 0)
+      (effects (font (size 1.27 1.27)) hide)
+    )
+    (property "MPN" "" (at 19.05 162.56 0)
+      (effects (font (size 1.27 1.27)) hide)
+    )
+    (property "Item #" "" (at 19.05 162.56 0)
+      (effects (font (size 1.27 1.27)) hide)
+    )
+    (property "Description" "" (at 19.05 162.56 0)
+      (effects (font (size 1.27 1.27)) hide)
+    )
+    (property "Package/Footprint" "" (at 19.05 162.56 0)
+      (effects (font (size 1.27 1.27)) hide)
+    )
+    (property "Type" "Thru-hole" (at 19.05 162.56 0)
+      (effects (font (size 1.27 1.27)) hide)
+    )
+    (property "Your Instructions / Notes" "" (at 19.05 162.56 0)
+      (effects (font (size 1.27 1.27)) hide)
+    )
+    (pin "1")
+    (pin "2")
+    (instances
+      (project "ble"
+        (path "/a75a1d04-4959-44a9-a64e-65228c5b9ff4"
+          (reference "J2") (unit 1)
+        )
+      )
